File: pcb_src/module/pmg001.sch (EAGLE design)
At the start: 42 parts, among them IC1 APX803D-29SAG-7, IC2 ATTINY1616-MNR, IC3 LD56100DPU30R, IC4 IP2312, IC5 TMP102AIDRLR, IC6 DMP3013SFV-7, IC9 INA219AIDCNR, U1 ADS1015IDGSR

Commit message: Module and cover board revised. Datasheet revised. Code added.
Updated with one additional component, added cutout to cover board. Updated documentation accordingly.  Added default program.
Parts:
- added Q1: PMZ290UNE2YL, edrtech_lib:PMZ290UNE2YL
- added R13: 20K, rcl:R-EU_R0402
- added R9: 150R, rcl:R-EU_R0402
Connections:
- new net N$1: Q1.G, R13.2, R9.2
- new net P_ON_DS: Q1.D, R14.1, R16.1
- net GND: now also Q1.S, R13.1
- net P_ON: now also R9.1; no longer R14.1, R16.1
Other:
- note added: "29.07.2024."
- note removed: "09.07.2024."
Changed lines of the file:
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@@
 <part name="U$1" library="edrtech_lib" deviceset="1.27_MALE_16P_HEADER" device=""/>
 <part name="U$2" library="edrtech_lib" deviceset="1.27_MALE_16P_HEADER" device=""/>
+<part name="Q1" library="edrtech_lib" deviceset="PMZ290UNE2YL" device=""/>
+<part name="R9" library="rcl" library_urn="urn:adsk.eagle:library:334" deviceset="R-EU_" device="R0402" package3d_urn="urn:adsk.eagle:package:23547/3" value="150R"/>
+<part name="R13" library="rcl" library_urn="urn:adsk.eagle:library:334" deviceset="R-EU_" device="R0402" package3d_urn="urn:adsk.eagle:package:23547/3" value="20K"/>
 </parts>
 <sheets>
@@
 <wire x1="92.71" y1="5.08" x2="13.97" y2="5.08" width="0.1524" layer="97"/>
 <text x="91.44" y="6.35" size="1.778" layer="97" align="bottom-right">EDRTECH D.O.O.</text>
-<text x="91.44" y="2.54" size="1.778" layer="97" align="bottom-right">09.07.2024.</text>
+<text x="91.44" y="2.54" size="1.778" layer="97" align="bottom-right">29.07.2024.</text>
 <wire x1="1.27" y1="12.7" x2="1.27" y2="182.88" width="0.1524" layer="97"/>
 <wire x1="1.27" y1="182.88" x2="299.72" y2="182.88" width="0.1524" layer="97"/>
@@
 <instance part="U$1" gate="G$1" x="27.94" y="53.34" smashed="yes"/>
 <instance part="U$2" gate="G$1" x="66.04" y="36.83" smashed="yes" rot="R180"/>
+<instance part="Q1" gate="G$1" x="86.36" y="74.93" smashed="yes">
+<attribute name="NAME" x="86.36" y="54.61" size="1.778" layer="95" rot="R90" align="center-left"/>
+<attribute name="VALUE" x="88.9" y="54.61" size="1.778" layer="96" rot="R90" align="center-left"/>
+</instance>
+<instance part="R9" gate="G$1" x="77.47" y="74.93" smashed="yes" rot="MR180">
+<attribute name="NAME" x="73.66" y="73.4314" size="1.778" layer="95" rot="MR180"/>
+<attribute name="VALUE" x="73.66" y="78.232" size="1.778" layer="96" rot="MR180"/>
+</instance>
+<instance part="R13" gate="G$1" x="83.82" y="67.31" smashed="yes" rot="MR90">
+<attribute name="NAME" x="85.3186" y="63.5" size="1.778" layer="95" rot="MR90"/>
+<attribute name="VALUE" x="80.518" y="63.5" size="1.778" layer="96" rot="MR90"/>
+</instance>
 </instances>
 <busses>
@@
 <label x="50.8" y="29.21" size="1.27" layer="95" rot="R270" xref="yes"/>
 <pinref part="U$2" gate="G$1" pin="P$7"/>
+</segment>
+<segment>
+<pinref part="Q1" gate="G$1" pin="S"/>
+<wire x1="93.98" y1="69.85" x2="93.98" y2="59.69" width="0.1524" layer="91"/>
+<label x="93.98" y="59.69" size="1.27" layer="95" rot="R270" xref="yes"/>
+</segment>
+<segment>
+<pinref part="R13" gate="G$1" pin="1"/>
+<wire x1="83.82" y1="62.23" x2="83.82" y2="59.69" width="0.1524" layer="91"/>
+<label x="83.82" y="59.69" size="1.27" layer="95" rot="R270" xref="yes"/>
 </segment>
 </net>
@@
 <net name="P_ON" class="0">
 <segment>
-<wire x1="96.52" y1="85.09" x2="93.98" y2="85.09" width="0.1524" layer="91"/>
-<wire x1="96.52" y1="92.71" x2="93.98" y2="92.71" width="0.1524" layer="91"/>
-<wire x1="93.98" y1="92.71" x2="93.98" y2="85.09" width="0.1524" layer="91"/>
-<wire x1="93.98" y1="85.09" x2="91.44" y2="85.09" width="0.1524" layer="91"/>
-<junction x="93.98" y="85.09"/>
-<label x="91.44" y="85.09" size="1.27" layer="95" rot="MR0" xref="yes"/>
-<pinref part="R14" gate="G$1" pin="1"/>
-<pinref part="R16" gate="G$1" pin="1"/>
-</segment>
-<segment>
 <pinref part="IC2" gate="G$1" pin="PA6"/>
 <wire x1="167.64" y1="26.67" x2="167.64" y2="24.13" width="0.1524" layer="91"/>
 <label x="167.64" y="24.13" size="1.27" layer="95" rot="R270" xref="yes"/>
+</segment>
+<segment>
+<pinref part="R9" gate="G$1" pin="1"/>
+<wire x1="72.39" y1="74.93" x2="69.85" y2="74.93" width="0.1524" layer="91"/>
+<label x="69.85" y="74.93" size="1.27" layer="95" rot="R180" xref="yes"/>
 </segment>
 </net>
@@
 </segment>
 </net>
+<net name="N$1" class="0">
+<segment>
+<pinref part="Q1" gate="G$1" pin="G"/>
+<pinref part="R9" gate="G$1" pin="2"/>
+<wire x1="86.36" y1="74.93" x2="83.82" y2="74.93" width="0.1524" layer="91"/>
+<pinref part="R13" gate="G$1" pin="2"/>
+<wire x1="83.82" y1="74.93" x2="82.55" y2="74.93" width="0.1524" layer="91"/>
+<wire x1="83.82" y1="72.39" x2="83.82" y2="74.93" width="0.1524" layer="91"/>
+<junction x="83.82" y="74.93"/>
+</segment>
+</net>
+<net name="P_ON_DS" class="0">
+<segment>
+<wire x1="96.52" y1="85.09" x2="93.98" y2="85.09" width="0.1524" layer="91"/>
+<wire x1="96.52" y1="92.71" x2="93.98" y2="92.71" width="0.1524" layer="91"/>
+<wire x1="93.98" y1="92.71" x2="93.98" y2="85.09" width="0.1524" layer="91"/>
+<wire x1="93.98" y1="85.09" x2="91.44" y2="85.09" width="0.1524" layer="91"/>
+<junction x="93.98" y="85.09"/>
+<label x="91.44" y="85.09" size="1.27" layer="95" rot="MR0" xref="yes"/>
+<pinref part="R14" gate="G$1" pin="1"/>
+<pinref part="R16" gate="G$1" pin="1"/>
+<pinref part="Q1" gate="G$1" pin="D"/>
+</segment>
+</net>
